File: NeatoXV11_Delta2G_adapter/NeatoXV11_Delta2G_adapter.kicad_pcb (KiCad board)
At the start: 2 copper layers, 43 x 21 mm, 10 parts, among them J1 JST PH B4B Vert, J2 JST PH B2B Vert, J3 JST PH B4B Vert, Q1 AS2302, U1 DNP LM2596

Commit message: Delta-2G
Parts:
- added J4: JST PH2.0 B5B Vert, Connector_JST:JST_PH_B5B-PH-K_1x05_P2.00mm_Vertical, F.Cu at (108.9, 45.1)
- J1: value JST PH B4B Vert -> JST PH2.0 B4B Vert
- J2: value JST PH B2B Vert -> JST PH2.0 B2B Vert
- moved Q1 0.25 mm to (105.5, 49.1)
Routing:
- net +5V: track 61.7 -> 85.9 mm
- net /TX: track 30.3 -> 43.7 mm
- net GND: track 93.4 -> 106.1 mm
- net /MOT+: track 16.3 -> 25.9 mm
- net /MOT-: track 9.38 -> 18.9 mm
Other:
- board text added: "D2 LDS"
- board text added: "Host MCU"
- board text added: "NX Motor NX Data"
- board text added: "NX-D2 LDS adapter board v0.3.0"
- board text removed: "Motor Data Laser distance sensor"
- board text removed: "NXVB LDS adapter board v0.2.0"
- board text removed: "To Host MCU"
