File: NeatoXV11_Delta2G_adapter/NeatoXV11_Delta2G_adapter.kicad_sch (KiCad schematic)
At the start: 10 parts, among them J1 JST PH B4B Vert, J2 JST PH B2B Vert, J3 JST PH B4B Vert, Q1 AS2302, U1 DNP LM2596

Commit message: Delta-2G
Parts:
- added J4: DNP JST PH2.0 B5B Vert, Connector_JST:JST_PH_B5B-PH-K_1x05_P2.00mm_Vertical, symbol Connector_Generic:Conn_01x05
- J1: value JST PH B4B Vert -> JST PH2.0 B4B Vert
- J2: value JST PH B2B Vert -> JST PH2.0 B2B Vert
Connections:
- net +5V: now also J4.3 (Pin_3)
- net GND: now also J4.2 (Pin_2)
- net MOT+: now also J4.5 (Pin_5)
- net MOT-: now also J4.4 (Pin_4)
- net TX: now also J4.1 (Pin_1)
Other:
- note added: "3irobotics Delta2G"
- title: Neato XV/Botvac LDS adapter -> Neato XV11/Delta-2G LDS adapter
- moved on the sheet: C1, D1, H1, H2, J1, J2, J3, JP1, Q1, U1
